Commit message: fix: patch改为标准a/b可git apply格式；修正arm_simple.urdf J4 rpy为3分量

File: stm32_arm/urdf/arm_simple.urdf (robot description, URDF)
Before this commit: robot six_dof_arm_simple, 7 links, 6 joints
Joints:
- joint joint4: origin xyz=0.047631 -0.1845 0 rpy=-1.5708 0 -> xyz=0.047631 -0.1845 0 rpy=-1.5708 0 0
